File: pcb/design.brd (EAGLE design)
At the start: 121.5 x 89 mm, 326 parts, among them IC1 TPS2065CDGNR, IC10 TPS2065CDGNR, IC2 SN74LVC1G126DCKR, IC3 SN74LVC1G126DCKR, IC4 TPS62111RSAR, IC5 CAT24C256YI-GT3, IC6 FT232RQ, IC7 EP5368QI, IC8 DNP, IC9 SN74LVC1G126DCKR, J1 10117836-002LF, J2 DF40C-100DS-0.4V(51), J3 10118192-0001LF, J4 7499111447, J5 DF40C-100DS-0.4V(51), J6 GSB311231HR, J7 70553-0002, J8 10117836-002LF, K1 CNU079S-008-A101, Q1 BSS138, Q2 FDN360P, Q3 FDN360P, Q4 BSS138, Q5 BSS138, U1 TPS5450QDDARQ1, U10 ASM1142, U11 TPS2052BDGNR, U12 67996-140HLF, U13 USB2513B-AEZG, U14 685 119 134 923, U15 USB5744/2G, U16 TPD4E02B04DQAR, U17 TPS5450QDDARQ1, U18 ADP1740ACPZ-1.2-R7, U19 TS3A5223RSWR, U2 TPD4E02B04DQAR, U20 TPD4E02B04DQAR, U21 TPD4E02B04DQAR, U22 TPD4E02B04DQAR, U23 TPD4E02B04DQAR, U24 TPS2066CDGNR, U3 TPD4E02B04DQAR, U4 TPD4E02B04DQAR, U5 TPD4E02B04DQAR, U6 TPD4E02B04DQAR, U7 TPD4E02B04DQAR, U8 TPD4E02B04DQAR, U9 TPD13S523PWR, Y1 ABM8G-24-18-D2Y-T, Y2 25.000MHz, Y3 ABM8G-20.000MHZ-18-D2Y-T

Commit message: pcb preliminary
Parts:
- C1: value C0603C0G1H470J030BA -> GRM0335C1E470JA01D; device qualified_1@eagle_src_repo_c6614e3cc11e779d3ff6357e0a9e972de604ed16:0201 -> qualified_1:0201
- C13, C262: value GRM31CR61H106KA12L -> CL31A106KBHNNNE
- C15, C299, C313, C65, C87: value GRM155R61A105KE01D -> CL05A105KO5NNNC
- C158, C167, C17, C25, C300, C34, C81, C89: value GRM185R60J475ME15D -> CGB3B1X5R1A475K055AC
- C19, C92: value CL21A226MQCLQNC -> 22uF
- C20, C21, C301, C302: value CC0201JRNPO9BN220 -> GRM0335C1H220JA01D
- C257, C261, C274, C305, C315, C316, C52, C78: value C0603X5R1A103K030BA -> GRM033R61C103KA12D
- C275, C3, C45, C46, C64: value C1608X5R0J106M080AB -> C1608X5R1A106M080AC
- C282, C283: value EMK107ABJ475KA-T -> C1608X5R1C475K080AC
- C285, C93: value UMK063CG100DTHF -> UMK063CG100DTF
- C319: value C0603C0G1H470J030BA -> GRM0335C1E470JA01D
- FB1, FB10, FB11, FB12, FB13, FB14, FB15, FB16, FB17, FB18, FB19, FB2, FB20, FB3, FB4, FB9: value BKP1005HM121-T -> BLM15PX121SN1D
- IC2, IC3, IC9: value SN74LVC1G126DCKR -> SN74LV1T126DCKR
- IC4: value TPS62111RSAR -> TPS62111RSAT
- IC6: value FT232RQ -> FT232RQ-REEL
- K1: value CNU079S-008-A101 -> 61400826021
- L14, L2: value IHLP3232DZER100M01 -> IHLP3232DZER100M11
- R1: device qualified_1@eagle_src_repo_c6614e3cc11e779d3ff6357e0a9e972de604ed16:0201 -> qualified_1:0201
- R12, R28, R30, R47, R5, R52, R53, R54, R59, R6, R63, R64, R7, R8: value CRCW0201100KFNED -> RC0201FR-07100KL
- R13, R20, R62: value RMCF0201FT1M00 -> 1M0
- R19: value RC0402JR-7D0RL -> RC1005J000CS
- R2: value ERJ-1GEF1500C -> ERJ-1GNJ151C; device qualified_1@eagle_src_repo_c6614e3cc11e779d3ff6357e0a9e972de604ed16:0201 -> qualified_1:0201
- R21, R3, R31, R39, R44, R49, R50, R60, R65, R69: value ERJ-1GE0R00C -> RC0201JR-070RL
- R24, R25: value RC0603F331CS -> ERJ-1GEJ331C
- R71: value ERJ-1GEF1500C -> ERJ-1GNJ151C
- S1: value EVQ-P7C01P -> EVQ-PLDA15; device qualified_1:EVQP-4 -> qualified_1:EVQ
- U14: value 685 119 134 923 -> 685119134923
- Y1: value ABM8G-24-18-D2Y-T -> ABM8G-24.000MHZ-18-D2Y-T
- Y2: value 25.000MHz -> ABM7-25.000MHZ-D2Y-T
- moved R1 12.6 mm to (13.3, 16.2), turned to 180 degrees
- moved D1 11.5 mm to (11.9, 17.3), turned to 90 degrees
- moved S1 10.7 mm to (11.8, 16.8), turned to 90 degrees
- moved R2 9.82 mm to (11.7, 16.1), turned to 0 degrees
- moved C1 7.86 mm to (10.3, 16.4), turned to 90 degrees
- moved D19 4.50 mm to (1.94, 13.4)
- moved C319 4.50 mm to (2.54, 17.0)
- moved R70 4.50 mm to (0.88, 16.7)
- moved R71 4.50 mm to (2.04, 16.1)
- moved S2 4.50 mm to (1.75, 15.0)
Connections:
- net 14.USB3_CC1_GPIO: now also C1.1, R2.2; no longer C319.1, R71.2
- net 14.nRESET_NRESET: now also C319.1, R71.2; no longer C1.1, R2.2
Routing:
- net GND: track 117.3 -> 119.6 mm, vias 205 -> 206
- net 14.USB3_CC1_GPIO: track 0.97 -> 2.00 mm, vias 0 -> 1
- net BTN_A$26: track 5.57 -> 4.72 mm
- net 14.VLOGIC_VLOGIC: track 10.4 -> 11.1 mm, vias 5 -> 6
