File: pcb/design.sch (EAGLE design)
At the start: 322 parts, among them IC1 TPS2065CDGNR, IC10 TPS2065CDGNR, IC2 SN74LVC1G126DCKR, IC3 SN74LVC1G126DCKR, IC4 TPS62111RSAR, IC5 CAT24C256YI-GT3, IC6 FT232RQ, IC7 EP5368QI, IC8 DNP, IC9 SN74LVC1G126DCKR, J1 10117836-002LF, J2 DF40C-100DS-0.4V(51), J3 10118192-0001LF, J4 7499111447, J5 DF40C-100DS-0.4V(51), J6 GSB311231HR, J7 70553-0002, J8 10117836-002LF, K1 CNU079S-008-A101, Q1 BSS138, Q2 FDN360P, Q3 FDN360P, Q4 BSS138, Q5 BSS138, U1 TPS5450QDDARQ1, U10 ASM1142, U11 TPS2052BDGNR, U12 67996-140HLF, U13 USB2513B-AEZG, U14 685 119 134 923, U15 USB5744/2G, U16 TPD4E02B04DQAR, U17 TPS5450QDDARQ1, U18 ADP1740ACPZ-1.2-R7, U19 TS3A5223RSWR, U2 TPD4E02B04DQAR, U20 TPD4E02B04DQAR, U21 TPD4E02B04DQAR, U22 TPD4E02B04DQAR, U23 TPD4E02B04DQAR, U24 TPS2066CDGNR, U3 TPD4E02B04DQAR, U4 TPD4E02B04DQAR, U5 TPD4E02B04DQAR, U6 TPD4E02B04DQAR, U7 TPD4E02B04DQAR, U8 TPD4E02B04DQAR, U9 TPD13S523PWR, Y1 ABM8G-24-18-D2Y-T, Y2 25.000MHz, Y3 ABM8G-20.000MHZ-18-D2Y-T

Commit message: pcb preliminary
Parts:
- C1: value C0603C0G1H470J030BA -> GRM0335C1E470JA01D; device qualified_1@eagle_src_repo_c6614e3cc11e779d3ff6357e0a9e972de604ed16:C0603C0G1H470J030BA -> qualified_1:GRM0335C1E470JA01D
- C13, C262: value GRM31CR61H106KA12L -> CL31A106KBHNNNE; device qualified_1@eagle_src_repo_f26ba765df9be4aea4dc36b2b99244de1327d3cb:GRM31CR61H106KA12L -> qualified_1@eagle_src_repo_f26ba765df9be4aea4dc36b2b99244de1327d3cb:CL31A106KBHNNNE
- C15, C299, C313: value GRM155R61A105KE01D -> CL05A105KO5NNNC; device qualified_1:GRM155R61A105KE01D -> qualified_1:CL05A105KO5NNNC
- C158, C167: value GRM185R60J475ME15D -> CGB3B1X5R1A475K055AC; device qualified_1@eagle_src_repo_701dee95a4f0c9d27f896634bd535ea9ef5a137e:GRM185R60J475ME15D -> qualified_1@eagle_src_repo_701dee95a4f0c9d27f896634bd535ea9ef5a137e:CGB3B1X5R1A475K055AC
- C17, C25, C34: value GRM185R60J475ME15D -> CGB3B1X5R1A475K055AC; device qualified_1@eagle_src_repo_b39d46a5feff4f7ade7f2a4f70c4d4847a03ea32:GRM185R60J475ME15D -> qualified_1@eagle_src_repo_b39d46a5feff4f7ade7f2a4f70c4d4847a03ea32:CGB3B1X5R1A475K055AC
- C19: value CL21A226MQCLQNC -> 22uF; device qualified_1@eagle_src_repo_b39d46a5feff4f7ade7f2a4f70c4d4847a03ea32:CL21A226MQCLQNC -> qualified_1@eagle_src_repo_b39d46a5feff4f7ade7f2a4f70c4d4847a03ea32:C0805
- C20, C21: value CC0201JRNPO9BN220 -> GRM0335C1H220JA01D; device qualified_1@eagle_src_repo_b39d46a5feff4f7ade7f2a4f70c4d4847a03ea32:CC0201JRNPO9BN220 -> qualified_1@eagle_src_repo_b39d46a5feff4f7ade7f2a4f70c4d4847a03ea32:GRM0335C1H220JA01D
- C257, C261: value C0603X5R1A103K030BA -> GRM033R61C103KA12D; device qualified_1@eagle_src_repo_08f38ff5c3a3a6fa35c93a02bac883b74ea519d0:C0603X5R1A103K030BA -> qualified_1@eagle_src_repo_08f38ff5c3a3a6fa35c93a02bac883b74ea519d0:GRM033R61C103KA12D
- C274: value C0603X5R1A103K030BA -> GRM033R61C103KA12D; device qualified_1@eagle_src_repo_8819a94826fe107100c913d4ec412d3185f90c61:C0603X5R1A103K030BA -> qualified_1@eagle_src_repo_8819a94826fe107100c913d4ec412d3185f90c61:GRM033R61C103KA12D
- C275: value C1608X5R0J106M080AB -> C1608X5R1A106M080AC; device qualified_1@eagle_src_repo_8819a94826fe107100c913d4ec412d3185f90c61:C1608X5R0J106M080AB -> qualified_1@eagle_src_repo_8819a94826fe107100c913d4ec412d3185f90c61:C1608X5R1A106M080AC
- C282, C283: value EMK107ABJ475KA-T -> C1608X5R1C475K080AC; device qualified_1@eagle_src_repo_701dee95a4f0c9d27f896634bd535ea9ef5a137e:EMK107ABJ475KA-T -> qualified_1@eagle_src_repo_701dee95a4f0c9d27f896634bd535ea9ef5a137e:C1608X5R1C475K080AC
- C285: value UMK063CG100DTHF -> UMK063CG100DTF; device qualified_1@eagle_src_repo_701dee95a4f0c9d27f896634bd535ea9ef5a137e:UMK063CG100DTHF -> qualified_1@eagle_src_repo_701dee95a4f0c9d27f896634bd535ea9ef5a137e:UMK063CG100DTF
- C3: value C1608X5R0J106M080AB -> C1608X5R1A106M080AC; device qualified_1@eagle_src_repo_d00aa7e5b0aed880e2479218df7f64b10b504166:C1608X5R0J106M080AB -> qualified_1@eagle_src_repo_d00aa7e5b0aed880e2479218df7f64b10b504166:C1608X5R1A106M080AC
- C300, C81, C89: value GRM185R60J475ME15D -> CGB3B1X5R1A475K055AC; device qualified_1:GRM185R60J475ME15D -> qualified_1:CGB3B1X5R1A475K055AC
- C301, C302: value CC0201JRNPO9BN220 -> GRM0335C1H220JA01D; device qualified_1:CC0201JRNPO9BN220 -> qualified_1:GRM0335C1H220JA01D
- C305: value C0603X5R1A103K030BA -> GRM033R61C103KA12D; device qualified_1@eagle_src_repo_d00aa7e5b0aed880e2479218df7f64b10b504166:C0603X5R1A103K030BA -> qualified_1@eagle_src_repo_d00aa7e5b0aed880e2479218df7f64b10b504166:GRM033R61C103KA12D
- C315, C316, C52, C78: value C0603X5R1A103K030BA -> GRM033R61C103KA12D; device qualified_1@eagle_src_repo_f26ba765df9be4aea4dc36b2b99244de1327d3cb:C0603X5R1A103K030BA -> qualified_1@eagle_src_repo_f26ba765df9be4aea4dc36b2b99244de1327d3cb:GRM033R61C103KA12D
- C319: value C0603C0G1H470J030BA -> GRM0335C1E470JA01D; device qualified_1@eagle_src_repo_c6614e3cc11e779d3ff6357e0a9e972de604ed16:C0603C0G1H470J030BA -> qualified_1@eagle_src_repo_c6614e3cc11e779d3ff6357e0a9e972de604ed16:GRM0335C1E470JA01D
- C45, C46: value C1608X5R0J106M080AB -> C1608X5R1A106M080AC; device qualified_1@eagle_src_repo_701dee95a4f0c9d27f896634bd535ea9ef5a137e:C1608X5R0J106M080AB -> qualified_1@eagle_src_repo_701dee95a4f0c9d27f896634bd535ea9ef5a137e:C1608X5R1A106M080AC
- C64: value C1608X5R0J106M080AB -> C1608X5R1A106M080AC; device qualified_1@eagle_src_repo_635c6cefb04d901352cb5cab0982b753f09e9156:C1608X5R0J106M080AB -> qualified_1@eagle_src_repo_635c6cefb04d901352cb5cab0982b753f09e9156:C1608X5R1A106M080AC
- C65: value GRM155R61A105KE01D -> CL05A105KO5NNNC; device qualified_1@eagle_src_repo_635c6cefb04d901352cb5cab0982b753f09e9156:GRM155R61A105KE01D -> qualified_1@eagle_src_repo_635c6cefb04d901352cb5cab0982b753f09e9156:CL05A105KO5NNNC
- C87: value GRM155R61A105KE01D -> CL05A105KO5NNNC; device qualified_1@eagle_src_repo_825e5973c79738778b249d35b895f4444d985c7a:GRM155R61A105KE01D -> qualified_1@eagle_src_repo_825e5973c79738778b249d35b895f4444d985c7a:CL05A105KO5NNNC
- C92: value CL21A226MQCLQNC -> 22uF; device qualified_1@eagle_src_repo_825e5973c79738778b249d35b895f4444d985c7a:CL21A226MQCLQNC -> qualified_1@eagle_src_repo_825e5973c79738778b249d35b895f4444d985c7a:C0805
- C93: value UMK063CG100DTHF -> UMK063CG100DTF; device qualified_1@eagle_src_repo_825e5973c79738778b249d35b895f4444d985c7a:UMK063CG100DTHF -> qualified_1@eagle_src_repo_825e5973c79738778b249d35b895f4444d985c7a:UMK063CG100DTF
- FB1, FB18, FB19, FB2, FB20, FB3: value BKP1005HM121-T -> BLM15PX121SN1D; device qualified_1@eagle_src_repo_0b5741b5d4abbb92614c593c71c49b300549e5ff:BKP1005HM121-T -> qualified_1@eagle_src_repo_0b5741b5d4abbb92614c593c71c49b300549e5ff:BLM15PX121SN1D
- FB10, FB11, FB12, FB13, FB14: value BKP1005HM121-T -> BLM15PX121SN1D; device qualified_1:BKP1005HM121-T -> qualified_1:BLM15PX121SN1D
- FB15, FB16, FB17, FB4: value BKP1005HM121-T -> BLM15PX121SN1D; device qualified_1@eagle_src_repo_d00aa7e5b0aed880e2479218df7f64b10b504166:BKP1005HM121-T -> qualified_1@eagle_src_repo_d00aa7e5b0aed880e2479218df7f64b10b504166:BLM15PX121SN1D
- FB9: value BKP1005HM121-T -> BLM15PX121SN1D; device qualified_1@eagle_src_repo_635c6cefb04d901352cb5cab0982b753f09e9156:BKP1005HM121-T -> qualified_1@eagle_src_repo_635c6cefb04d901352cb5cab0982b753f09e9156:BLM15PX121SN1D
- IC2, IC9: value SN74LVC1G126DCKR -> SN74LV1T126DCKR; device qualified_1:SN74LVC1G126DCKRAHC -> qualified_1:SN74LV1T126DCKRAHC
- IC3: value SN74LVC1G126DCKR -> SN74LV1T126DCKR; device qualified_1:SN74LVC1G126DCKR -> qualified_1:SN74LV1T126DCKR
- IC4: value TPS62111RSAR -> TPS62111RSAT; device qualified_1:TPS62111RSAR -> qualified_1:TPS62111RSAT
- IC6: value FT232RQ -> FT232RQ-REEL; device qualified_1:FT232RQ -> qualified_1:FT232RQ-REEL
- K1: value CNU079S-008-A101 -> 61400826021; device qualified_1:CNU079S-008-A101 -> qualified_1:61400826021
- L14, L2: value IHLP3232DZER100M01 -> IHLP3232DZER100M11; device qualified_1@eagle_src_repo_f26ba765df9be4aea4dc36b2b99244de1327d3cb:IHLP3232DZER100M01 -> qualified_1@eagle_src_repo_f26ba765df9be4aea4dc36b2b99244de1327d3cb:IHLP3232DZER100M11
- R1: device qualified_1@eagle_src_repo_c6614e3cc11e779d3ff6357e0a9e972de604ed16:RC0201FR-0710KL -> qualified_1:RC0201FR-0710KL
- R12, R59: value CRCW0201100KFNED -> RC0201FR-07100KL; device qualified_1@eagle_src_repo_f26ba765df9be4aea4dc36b2b99244de1327d3cb:CRCW0201100KFNED -> qualified_1@eagle_src_repo_f26ba765df9be4aea4dc36b2b99244de1327d3cb:RC0201FR-07100KL
- R13, R62: value RMCF0201FT1M00 -> 1M0; device qualified_1:RMCF0201FT1M00 -> qualified_1:R0201
- R19: value RC0402JR-7D0RL -> RC1005J000CS; device qualified_1@eagle_src_repo_825e5973c79738778b249d35b895f4444d985c7a:RC0402JR-7D0RL -> qualified_1@eagle_src_repo_825e5973c79738778b249d35b895f4444d985c7a:RC1005J000CS
- R2: value ERJ-1GEF1500C -> ERJ-1GNJ151C; device qualified_1@eagle_src_repo_c6614e3cc11e779d3ff6357e0a9e972de604ed16:ERJ-1GEF1500C -> qualified_1:ERJ-1GNJ151C
- R20: value RMCF0201FT1M00 -> 1M0; device qualified_1@eagle_src_repo_825e5973c79738778b249d35b895f4444d985c7a:RMCF0201FT1M00 -> qualified_1@eagle_src_repo_825e5973c79738778b249d35b895f4444d985c7a:R0201
- R21: value ERJ-1GE0R00C -> RC0201JR-070RL; device qualified_1@eagle_src_repo_825e5973c79738778b249d35b895f4444d985c7a:ERJ-1GE0R00C -> qualified_1@eagle_src_repo_825e5973c79738778b249d35b895f4444d985c7a:RC0201JR-070RL
- R24, R25: value RC0603F331CS -> ERJ-1GEJ331C; device qualified_1@eagle_src_repo_635c6cefb04d901352cb5cab0982b753f09e9156:RC0603F331CS -> qualified_1@eagle_src_repo_635c6cefb04d901352cb5cab0982b753f09e9156:ERJ-1GEJ331C
- R28, R30, R47, R5, R52, R53, R54, R6, R63, R64, R7, R8: value CRCW0201100KFNED -> RC0201FR-07100KL; device qualified_1:CRCW0201100KFNED -> qualified_1:RC0201FR-07100KL
- R3, R31, R44, R49, R50, R60, R65, R69: value ERJ-1GE0R00C -> RC0201JR-070RL; device qualified_1:ERJ-1GE0R00C -> qualified_1:RC0201JR-070RL
- R39: value ERJ-1GE0R00C -> RC0201JR-070RL; device qualified_1@eagle_src_repo_83354d0c2c11c8ce792d5cc032a7091e5ff73f00:ERJ-1GE0R00C -> qualified_1@eagle_src_repo_83354d0c2c11c8ce792d5cc032a7091e5ff73f00:RC0201JR-070RL
- R71: value ERJ-1GEF1500C -> ERJ-1GNJ151C; device qualified_1@eagle_src_repo_c6614e3cc11e779d3ff6357e0a9e972de604ed16:ERJ-1GEF1500C -> qualified_1@eagle_src_repo_c6614e3cc11e779d3ff6357e0a9e972de604ed16:ERJ-1GNJ151C
- S1: value EVQ-P7C01P -> EVQ-PLDA15; device qualified_1:EVQ-P7C01P -> qualified_1:EVQ-PLDA15
- U14: value 685 119 134 923 -> 685119134923; device qualified_1:685-119-134-923 -> qualified_1:685119134923
- Y1: value ABM8G-24-18-D2Y-T -> ABM8G-24.000MHZ-18-D2Y-T; device qualified_1:ABM8G-24-18-D2Y-T -> qualified_1:ABM8G-24.000MHZ-18-D2Y-T
- Y2: value 25.000MHz -> ABM7-25.000MHZ-D2Y-T; device qualified_1@eagle_src_repo_b39d46a5feff4f7ade7f2a4f70c4d4847a03ea32:X2CS10 -> qualified_1@eagle_src_repo_b39d46a5feff4f7ade7f2a4f70c4d4847a03ea32:ABM7-25.000MHZ-D2Y-T
Connections:
- net 14.USB3_CC1_GPIO: now also C1.1, R2.2; no longer C319.1, R71.2
- net 14.nRESET_NRESET: now also C319.1, R71.2; no longer C1.1, R2.2
Other:
- note added: "24) Pushbutton"
- note added: "HurraCloud v0.4"
- note added: "Pushbutton"
- note removed: "24) Pushbutton R/A"
- note removed: "HurraCloud v0.3"
